File: schematics/ATTinyProgrammingShield.kicad_pcb (KiCad board)
At the start: 2 copper layers, 55.9 x 34.3 mm, 6 parts, among them J1 DIP8_Socket, J2 Conn_01x08_Male, J3 Conn_01x10_Male

Commit message: Update to KiCad 5 from KiCad 4
- use KiCad's standard library Arduino shield symbol and footprint
- ground the second copper layer of the PCB (and consequently unground
the first copper layer of the PCB)
Routing:
- added copper zone on B.Cu, net Earth
- removed copper zone on F.Cu, net Earth
Changed lines of the file:
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@@
-(kicad_pcb (version 4) (host pcbnew 4.0.7-e2-6376~61~ubuntu18.04.1)
+(kicad_pcb (version 20171130) (host pcbnew 5.0.0-fee4fd1~65~ubuntu18.04.1)
   (general
-    (links 11)
-    (no_connects 0)
-    (area 125.187142 68.504999 187.232858 102.945001)
     (thickness 1.6)
     (drawings 33)
@@
       (layerselection 0x010f0_80000001)
       (usegerberextensions false)
+      (usegerberattributes false)
+      (usegerberadvancedattributes false)
+      (creategerberjobfile false)
       (excludeedgelayer true)
       (linewidth 0.100000)
@@
       (hpglpennumber 1)
       (hpglpenspeed 20)
-      (hpglpendiameter 15)
-      (hpglpenoverlay 2)
+      (hpglpendiameter 15.000000)
       (psnegative false)
       (psa4output false)
@@
       (drillshape 0)
       (scaleselection 1)
-      (outputdirectory gerber/))
+      (outputdirectory "gerber/"))
   )
   (net 0 "")
@@
     (fp_line (start 1.8 -19.55) (end 1.8 1.8) (layer B.CrtYd) (width 0.05))
     (fp_line (start 1.8 1.8) (end -1.8 1.8) (layer B.CrtYd) (width 0.05))
-    (fp_text user %R (at 0 -8.89 450) (layer B.Fab)
+    (fp_text user %R (at 0 -8.89 90) (layer B.Fab)
       (effects (font (size 1 1) (thickness 0.15)) (justify mirror))
     )
@@
     (fp_line (start 1.8 -24.65) (end 1.8 1.8) (layer B.CrtYd) (width 0.05))
     (fp_line (start 1.8 1.8) (end -1.8 1.8) (layer B.CrtYd) (width 0.05))
-    (fp_text user %R (at 0 -11.43 450) (layer B.Fab)
+    (fp_text user %R (at 0 -11.43 90) (layer B.Fab)
       (effects (font (size 1 1) (thickness 0.15)) (justify mirror))
     )
@@
   (segment (start 140.462 89.154) (end 132.08 89.154) (width 0.25) (layer F.Cu) (net 10) (status 20))
   (segment (start 148.336 81.28) (end 140.462 89.154) (width 0.25) (layer F.Cu) (net 10))
-  (zone (net 2) (net_name Earth) (layer F.Cu) (hatch edge 0.508)
-    (connect_pads (clearance 0.508))
-    (min_thickness 0.254)
-    (fill yes (arc_segments 16) (thermal_gap 0.508) (thermal_bridge_width 0.508))
-    (polygon
-      (pts
-        (xy 184.15 102.87) (xy 128.27 102.87) (xy 128.27 68.58) (xy 184.15 68.58)
-      )
-    )
-  )
   (zone (net 0) (net_name "") (layer F.SilkS) (hatch edge 0.508)
     (connect_pads (clearance 0.508))
@@
       )
     )
+  )
+  (zone (net 2) (net_name Earth) (layer B.Cu) (hatch edge 0.508)
+    (connect_pads (clearance 0.508))
+    (min_thickness 0.254)
+    (fill yes (arc_segments 16) (thermal_gap 0.508) (thermal_bridge_width 0.508))
+    (polygon
+      (pts
+        (xy 184.15 68.58) (xy 184.15 102.87) (xy 128.27 102.87) (xy 128.27 68.58)
+      )
+    )
